File: Q930.kicad_pcb (KiCad board)
At the start: 2 copper layers, 2 parts, among them U1 MW-R-WX

Commit message: continue
Parts:
- added LED1: LB Q39E-L2OO-35-1, q930:LED_LBQ39E_OSR, F.Cu at (154.2, 79.4)
- added U2: DRV5032FDDMRR, q930:DMR0004A, F.Cu at (153.8, 75.3)
- added U3: SHT40I-AD1B-R2, q930:SHT40I_SEN, F.Cu at (150.3, 79.7)
- added U4: TPL5010DDCR, q930:DDC0006A_N, F.Cu at (150.1, 76.0)
Connections:
- net Net-(BT1-+) renamed +3V0
- U1 pad 14: unconnected-(U1-DIO14/SCL-Pad14) -> W_SCL
- U1 pad 17: unconnected-(U1-DIO15/SDA-Pad17) -> W_SDA
- U1 pad 2: unconnected-(U1-DO1/PWM3-Pad2) -> Net-(J1-Pin_3)
- U1 pad 21: unconnected-(U1-~{RESET}-Pad21) -> Net-(J1-Pin_5)
- U1 pad 7: unconnected-(U1-DIO5/PWM1-Pad7) -> LED
- U1 pad 8: unconnected-(U1-DIO6/TX-Pad8) -> Net-(J1-Pin_2)
- U1 pad 9: unconnected-(U1-DIO7/RX-Pad9) -> Net-(J1-Pin_4)

Commit message: 途中
Parts:
- added C1: 0.1u, Capacitor_SMD:C_0603_1608Metric_Pad1.08x0.95mm_HandSolder, F.Cu at (161.2, 108.5)
- added C2: 0.1u, Capacitor_SMD:C_0603_1608Metric_Pad1.08x0.95mm_HandSolder, F.Cu at (161.2, 111.1)
- added C3: 0.1u, Capacitor_SMD:C_0603_1608Metric_Pad1.08x0.95mm_HandSolder, F.Cu at (161.2, 113.6)
- added D1: 1SS387CT_L3FT, q930:CST2_TOS, F.Cu at (146.9, 101.2)
- added R1: 3.3k, Resistor_SMD:R_0201_0603Metric_Pad0.64x0.40mm_HandSolder, F.Cu at (164.8, 108.2)
- added R2: 3.3k, Resistor_SMD:R_0201_0603Metric_Pad0.64x0.40mm_HandSolder, F.Cu at (164.8, 109.9)
- added R3: 470, Resistor_SMD:R_0201_0603Metric_Pad0.64x0.40mm_HandSolder, F.Cu at (164.8, 111.7)
- added R4: 27k, Resistor_SMD:R_0201_0603Metric_Pad0.64x0.40mm_HandSolder, F.Cu at (164.8, 113.4)
- U4: footprint q930:DDC0006A_N -> q930:DDC0006A_L
- moved U4 17.8 mm to (133.8, 83.1)
- moved U3 9.38 mm to (155.0, 87.9)
Connections:
- U1 pad 15: unconnected-(U1-DIO13/DI2-Pad15) -> WDTOUT
- U1 pad 21: Net-(J1-Pin_5) -> RESETN
- U4 pad 4: unconnected-(U4-DONE-Pad4) -> WDTOUT
- U4 pad 6: unconnected-(U4-RST_N-Pad6) -> Net-(U4-RST_N)

Commit message: 途中
Parts:
- added J1: 7Pin, Connector_PinSocket_2.54mm:PinSocket_1x07_P2.54mm_Vertical_SMD_Pin1Left, F.Cu at (146.3, 47.0)
- added U5: SEN-14480, q930:SEN-14480, F.Cu at (117.5, 99.7)
- BT1: value Battery_Cell -> CR2032
- moved BT1 27.4 mm to (118.0, 99.7)
Connections:
- net LED renamed /LED
- net WDTOUT renamed /WDTOUT
- U1 pad 10: unconnected-(U1-DIO8/PWM4-Pad10) -> /SNS_OUT2
- U1 pad 13: unconnected-(U1-DIO12/DI1-Pad13) -> Net-(J1-Pin_7)
- U1 pad 18: unconnected-(U1-DIO16/DI4-Pad18) -> /SNS_OUT1
- U1 pad 2: Net-(J1-Pin_3) -> /SPIMISO
- U1 pad 24: unconnected-(U1-DIO0/AI2-Pad24) -> /INT1
- U1 pad 25: unconnected-(U1-DIO1/AI4-Pad25) -> /INT2
- U1 pad 8: Net-(J1-Pin_2) -> /TX
- U1 pad 9: Net-(J1-Pin_4) -> /RX
- U2 pad 3: SNS_OUT2 -> /SNS_OUT2
- U2 pad 4: SNS_OUT1 -> /SNS_OUT1
